File: SAM-simplified/SAM4/connections.kicad_sch (KiCad schematic)
At the start: 6 parts, among them J1 Conn_01x02_Pin, J10 Conn_01x02_Female, J6 XT60PW-M, J7 XT60PW-M, J8 XT30PW-F, SW1 SW_SPST

Commit message: add production files for EasyLAM PDB, STEP for EasySAM
Parts:
- J1: footprint (none) -> Connector_PinHeader_2.54mm:PinHeader_1x02_P2.54mm_Horizontal
Changed lines of the file:
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@@
 			)
 		)
-		(property "Footprint" ""
+		(property "Footprint" "Connector_PinHeader_2.54mm:PinHeader_1x02_P2.54mm_Horizontal"
 			(at 168.91 26.67 0)
 			(effects
